Commit message: revise origin to fit robot model and pointcloud

File: 05-pick-n-place/02-UR3/pickathon/src/robot_description/urdf/ur3_real.urdf.xacro (robot description, xacro)
@@ -321,5 +321,5 @@
     </link>
     <joint name="${prefix}camera_fixed_joint" type="fixed">
-      <origin xyz="0 -0.074 0" rpy="${pi/2} 0 0"/>
+      <origin xyz="0.014 -0.06 0.004" rpy="${pi/2} 0 0"/>
       <parent link="${prefix}ee_link"/>
       <child link="camera_link"/>
